Commit message: Rezolvat TF tree base_link, corectat URDF și adăugat configurare SLAM Toolbox

File: install/turtlebot_description/share/turtlebot_description/urdf/robot.urdf.xacro (robot description, xacro)
@@ -5,7 +5,7 @@
     <material name="blue"><color rgba="0.2 0.2 0.8 1"/></material>
     <!-- LINK DE BAZĂ -->
-    <link name="base_footprint"/>
+    <link name="base_link"/>
     <joint name="base_joint" type="fixed">
-        <parent link="base_footprint"/>
+        <parent link="base_link"/>
         <child link="chassis"/>
         <origin xyz="0 0 0.05" rpy="0 0 0"/>
@@ -119,5 +119,5 @@
             <tf_topic>/tf</tf_topic>
             <frame_id>odom</frame_id>
-            <child_frame_id>base_footprint</child_frame_id>
+            <child_frame_id>base_link</child_frame_id>
             <odom_publish_frequency>30</odom_publish_frequency>
         </plugin>

Commit message: Rezolvat comenzi tasatatura si viteza roti

File: install/turtlebot_description/share/turtlebot_description/urdf/robot.urdf.xacro (robot description, xacro)
@@ -53,5 +53,5 @@
         <parent link="chassis"/>
         <child link="right_wheel"/>
-        <origin xyz="0.04 -0.08 0" rpy="1.5708 0 0"/>
+        <origin xyz="0.04 -0.08 0" rpy="-1.5708 0 0"/>
         <axis xyz="0 0 1"/>
     </joint>
